File: main-esp-breakout-board.kicad_sch (KiCad schematic)
At the start: 0 parts

Commit message: finished rudimentary schematic; still needs review and PCB layout...
Parts:
- added C1, C13: 10uf, Capacitor_THT:CP_Radial_D5.0mm_P2.50mm, symbol Device:C_Polarized
- added C10, C11, C12, C3, C4, C5, C6, C7, C8, C9: 1nF, Capacitor_THT:C_Disc_D5.0mm_W2.5mm_P2.50mm, symbol Device:C
- added C2: 1uf, Capacitor_THT:CP_Radial_D5.0mm_P2.50mm, symbol Device:C_Polarized
- added D1, D3, D4, D5, D6, D7, D8: 3V3, Diode_THT:D_DO-15_P5.08mm_Vertical_KathodeUp, symbol Device:D_Zener
- added J1, J4, J_arm_motor_signals2, J_switch_0, J_switch_1, J_switch_2, J_switch_3, J_switch_4, J_switch_5, J_switch_6, J_switch_7: Conn_01x02_Socket, Connector_PinHeader_2.54mm:PinHeader_1x02_P2.54mm_Vertical, symbol Connector:Conn_01x02_Socket
- added J2, J3: Conn_01x18_Pin, Connector_PinHeader_2.54mm:PinHeader_1x18_P2.54mm_Vertical, symbol Connector:Conn_01x18_Pin
- added J_arm_motor_signals1, J_arm_pots1, J_encoder_1, J_encoder_2, J_encoder_3, J_encoder_4, J_i2c_1, J_i2c_2, J_i2c_3, J_ir_beac_a1, J_ir_beac_b1, J_reflectance_1: Conn_01x05_Socket, Connector_PinSocket_2.54mm:PinSocket_1x05_P2.54mm_Vertical, symbol Connector:Conn_01x05_Socket
- added J_hbridge_1, J_hbridge_2, J_hbridge_3, J_hbridge_4: Conn_01x03_Socket, Connector_PinSocket_2.54mm:PinSocket_1x03_P2.54mm_Vertical, symbol Connector:Conn_01x03_Socket
- added Q1, Q10, Q11, Q2, Q3, Q4, Q5, Q6, Q7, Q8, Q9: 2N3904, Package_TO_SOT_THT:TO-92_Inline, symbol Transistor_BJT:2N3904
- added R1: 4.7k, Resistor_THT:R_Axial_DIN0204_L3.6mm_D1.6mm_P2.54mm_Vertical, symbol Device:R
- added R10, R12, R14, R16, R18, R20, R22, R24, R26, R28, R30: 100k, symbol Device:R
- added R11, R13, R15, R17, R19, R21, R23, R25, R27, R29, R31: 10k, symbol Device:R
- added R2, R3, R4, R5, R6, R7, R8, R9: 4.7k, Resistor_THT:R_Axial_DIN0204_L3.6mm_D1.6mm_P1.90mm_Vertical, symbol Device:R
- added R4.7k: R, Resistor_THT:R_Axial_DIN0204_L3.6mm_D1.6mm_P2.54mm_Vertical, symbol Device:R
- added U1: ~, Project_Lib:Untitled, symbol project_lib:esp32_pico
- added U2: MC33269T-3.3, Project_Lib:TO220-3_ONS, symbol project_lib:MC33269T-3.3
- added U3: CD4051B, symbol Analog_Switch:CD4051B
- added U4, U5: CD74HC4094E, N16, symbol shift_reg:CD74HC4094E
- added U6: CD4053B, symbol Analog_Switch:CD4053B
Connections:
- new net: Q2.3 (C), R13.1, U3.10 (B)
- new net: Q9.2 (B), R26.2
- new net: J_hbridge_4.1 (Pin_1), Q9.3 (C), R27.1
- new net: J_switch_7.2 (Pin_2), R9.2
- new net: J_arm_motor_signals1.3 (Pin_3), Q11.3 (C), R31.1
- new net: J_switch_4.2 (Pin_2), R6.2
- new net: J_arm_motor_signals1.1 (Pin_1), Q10.3 (C), R29.1
- new net: J_switch_2.2 (Pin_2), R4.2
- new net: Q6.2 (B), R20.2
- new net: J_hbridge_1.1 (Pin_1), Q6.3 (C), R21.1
- new net: Q5.3 (C), R19.1
- new net: Q7.2 (B), R22.2
- new net: J_hbridge_2.1 (Pin_1), Q7.3 (C), R23.1
- new net: Q11.2 (B), R30.2
- new net: Q1.2 (B), R10.2
- new net: Q1.3 (C), R11.1, U3.11 (A)
- new net: Q8.2 (B), R24.2
- new net: Q4.3 (C), R17.1, U6.10 (S2), U6.11 (S1), U6.9 (S3)
- new net: Q3.2 (B), R14.2
- new net: J_hbridge_3.1 (Pin_1), Q8.3 (C), R25.1
- new net: Q5.2 (B), R18.2
- new net: J_switch_3.2 (Pin_2), R5.2
- new net: Q2.2 (B), R12.2
- new net: J_switch_0.2 (Pin_2), R2.2
- new net: J_switch_6.2 (Pin_2), R8.2
- new net: J_switch_5.2 (Pin_2), R7.2
- new net: Q3.3 (C), R15.1, U3.9 (C)
- new net: U4.10 (QS2), U5.2 (DATA)
- new net: J_switch_1.2 (Pin_2), R3.2
- new net: Q4.2 (B), R16.2
- new net: Q10.2 (B), R28.2
- new net +5V: C13.1, C2.1, J3.18 (Pin_18), J4.1 (Pin_1), J_encoder_1.5 (Pin_5), J_i2c_1.5 (Pin_5), J_i2c_2.5 (Pin_5), J_i2c_3.5 (Pin_5), J_reflectance_1.1 (Pin_1), R11.2, R13.2, R15.2, R17.2, U1.41 (5V), U2.3 (VIN), U3.16 (VDD), U6.16 (VDD)
- new net 0: J3.15 (Pin_15), J_encoder_4.3 (Pin_3), U1.0 (gpio_0)
- new net 1: J_hbridge_4.2 (Pin_2)
- new net 10: J2.11 (Pin_11), J2.8 (Pin_8), J_hbridge_1.2 (Pin_2), U1.1 (gpio_1), U1.10 (gpio_10)
- new net 12: J3.10 (Pin_10), J_encoder_2.2 (Pin_2), U1.12 (gpio_12)
- new net 13: J3.11 (Pin_11), J_encoder_2.3 (Pin_3), U1.13 (gpio_13)
- new net 14: J3.9 (Pin_9), J_encoder_1.3 (Pin_3), U1.14 (gpio_14)
- new net 15: J3.12 (Pin_12), J_encoder_3.2 (Pin_2), U1.15 (gpio_15)
- new net 19: J2.4 (Pin_4), U1.19 (gpio_19), U4.1 (STROBE), U5.1 (STROBE)
- new net 2: J3.13 (Pin_13), J_encoder_3.3 (Pin_3), U1.2 (gpio_2)
- new net 20: D1.1 (K), J2.1 (Pin_1), U1.20 (gpio_20), U3.3 (X)
- new net 21: J2.2 (Pin_2), U1.21 (gpio_21), U4.2 (DATA)
- new net 22: J2.3 (Pin_3), U1.22 (gpio_22), U4.3 (CP), U5.3 (CP)
- new net 25: J3.4 (Pin_4), J_i2c_1.1 (Pin_1), J_i2c_2.1 (Pin_1), J_i2c_3.1 (Pin_1), R1.1, U1.25 (gpio_25)
- new net 26: J3.5 (Pin_5), J_i2c_1.2 (Pin_2), J_i2c_2.2 (Pin_2), J_i2c_3.2 (Pin_2), R4.7k.1, U1.26 (gpio_26)
- new net 27: J3.8 (Pin_8), J_encoder_1.2 (Pin_2), U1.27 (gpio_27)
- new net 3: J2.10 (Pin_10), J_hbridge_3.2 (Pin_2), U1.3 (gpio_3)
- new net 32: D4.1 (K), J3.6 (Pin_6), J_arm_pots1.2 (Pin_2), U1.32 (gpio_32)
- new net 33: D5.1 (K), J3.7 (Pin_7), J_arm_pots1.3 (Pin_3), U1.33 (gpio_33)
- new net 34: D7.1 (K), J2.13 (Pin_13), U1.34 (gpio_34), U6.15 (B)
- new net 35: D6.1 (K), J2.12 (Pin_12), U1.35 (gpio_35), U6.14 (A)
- new net 36: D3.1 (K), J3.2 (Pin_2), J_reflectance_1.3 (Pin_3), U1.36 (gpio_36)
- new net 37: J2.15 (Pin_15), J_arm_motor_signals2.1 (Pin_1), U1.37 (gpio_37)
- new net 38: J2.14 (Pin_14), U1.38 (gpio_38), U6.4 (C)
- new net 39: D8.1 (K), J3.3 (Pin_3), J_reflectance_1.4 (Pin_4), U1.39 (gpio_39)
- new net 4: J3.14 (Pin_14), J_encoder_4.2 (Pin_2), U1.4 (gpio_4)
- new net 5: J2.7 (Pin_7), J_arm_motor_signals1.5 (Pin_5), U1.5 (gpio_5)
- new net 7: J2.6 (Pin_6), J_arm_motor_signals1.4 (Pin_4), U1.7 (gpio_7)
- new net 8: J2.5 (Pin_5), J_arm_motor_signals1.2 (Pin_2), U1.8 (gpio_8)
- new net 9: J2.9 (Pin_9), J_hbridge_2.2 (Pin_2), U1.9 (gpio_9)
- new net CHIP_PU: J2.16 (Pin_16), U1.43 (CHIP_PU)
- new net GND: C1.2, C10.2, C11.1, C12.1, C13.2, C2.2, C3.2, C4.2, C5.2, C6.2, C7.2, C8.2, C9.2, D1.2 (A), D3.2 (A), D4.2 (A), D5.2 (A), D6.2 (A), D7.2 (A), D8.2 (A), J1.2 (Pin_2), J2.17 (Pin_17), J3.1 (Pin_1), J3.17 (Pin_17), J4.2 (Pin_2), J_arm_motor_signals2.2 (Pin_2), J_arm_pots1.5 (Pin_5), J_encoder_1.4 (Pin_4), J_encoder_2.4 (Pin_4), J_encoder_3.4 (Pin_4), J_encoder_4.4 (Pin_4), J_hbridge_1.3 (Pin_3), J_hbridge_2.3 (Pin_3), J_hbridge_3.3 (Pin_3), J_hbridge_4.3 (Pin_3), J_i2c_1.3 (Pin_3), J_i2c_2.3 (Pin_3), J_i2c_3.3 (Pin_3), J_ir_beac_a1.5 (Pin_5), J_ir_beac_b1.5 (Pin_5), J_reflectance_1.5 (Pin_5), Q1.1 (E), Q10.1 (E), Q11.1 (E), Q2.1 (E), Q3.1 (E), Q4.1 (E), Q5.1 (E), Q6.1 (E), Q7.1 (E), Q8.1 (E), Q9.1 (E), U1.40 (GND), U2.1 (GND/ADJ), U3.6 (INH), U3.7 (VEE), U3.8 (VSS), U4.8 (GND), U5.8 (GND), U6.6 (INH), U6.7 (VEE), U6.8 (VSS)
- new net IR_BEAC_1A: J_ir_beac_a1.2 (Pin_2), U6.12 (A0)
- new net IR_BEAC_1B: J_ir_beac_b1.2 (Pin_2), U6.13 (A1)
- new net IR_BEAC_2A: J_ir_beac_a1.3 (Pin_3), U6.2 (B0)
- new net IR_BEAC_2B: J_ir_beac_b1.3 (Pin_3), U6.1 (B1)
- new net IR_BEAC_SERV_A: J_ir_beac_a1.4 (Pin_4), U6.5 (C0)
- new net IR_BEAC_SERV_B: J_ir_beac_b1.4 (Pin_4), U6.3 (C1)
- new net SHIFT_0: R20.1, U4.4 (Q0)
- new net SHIFT_1: R22.1, U4.5 (Q1)
- new net SHIFT_10: R14.1, U5.6 (Q2)
- new net SHIFT_11: R16.1, U5.7 (Q3)
- new net SHIFT_12: U5.14 (Q4)
- new net SHIFT_13: U5.13 (Q5)
- new net SHIFT_14: U5.12 (Q6)
- new net SHIFT_15: U5.11 (Q7)
- new net SHIFT_2: R24.1, U4.6 (Q2)
- new net SHIFT_3: R26.1, U4.7 (Q3)
- new net SHIFT_4: R28.1, U4.14 (Q4)
- new net SHIFT_5: R30.1, U4.13 (Q5)
- new net SHIFT_6: U4.12 (Q6)
- new net SHIFT_7: U4.11 (Q7)
- new net SHIFT_8: R10.1, U5.4 (Q0)
- new net SHIFT_9: R12.1, U5.5 (Q1)
- new net S_MUX_0: C3.1, R2.1, U3.13 (X0)
- new net S_MUX_1: C4.1, R3.1, U3.14 (X1)
- new net S_MUX_2: C5.1, R4.1, U3.15 (X2)
- new net S_MUX_3: C6.1, R5.1, U3.12 (X3)
- new net S_MUX_4: C7.1, R6.1, U3.1 (X4)
- new net S_MUX_5: C8.1, R7.1, U3.5 (X5)
- new net S_MUX_6: C9.1, R8.1, U3.2 (X6)
- new net S_MUX_7: C10.1, R9.1, U3.4 (X7)
- new net esp_3.3: J2.18 (Pin_18), J3.16 (Pin_16), U1.42 (3V3)
- new net supply_3.3: C1.1, C11.2, C12.2, J_arm_pots1.1 (Pin_1), J_encoder_1.1 (Pin_1), J_i2c_1.4 (Pin_4), J_i2c_2.4 (Pin_4), J_i2c_3.4 (Pin_4), J_ir_beac_a1.1 (Pin_1), J_ir_beac_b1.1 (Pin_1), J_reflectance_1.2 (Pin_2), J_switch_0.1 (Pin_1), J_switch_1.1 (Pin_1), J_switch_2.1 (Pin_1), J_switch_3.1 (Pin_1), J_switch_4.1 (Pin_1), J_switch_5.1 (Pin_1), J_switch_6.1 (Pin_1), J_switch_7.1 (Pin_1), R1.2, R19.2, R21.2, R23.2, R25.2, R27.2, R29.2, R31.2, R4.7k.2, U2.2 (VOUT), U4.15 (OE), U4.16 (VCC), U5.15 (OE), U5.16 (VCC)
Other:
- note added: "3.3V regulator to power sensors."
- note added: "Arm Pot Connections"
- note added: "Encoder Connections"
- note added: "I2C"
- note added: "Input from Buck Regulator."
- note added: "Reflectance Sensor"
- note added: "Shoulder Dir"
- note added: "Turntable Dir"

Commit message: halfway thru layout...
Parts:
- removed J1, J_arm_motor_signals2: Conn_01x02_Socket, Connector_PinHeader_2.54mm:PinHeader_1x02_P2.54mm_Vertical, symbol Connector:Conn_01x02_Socket
- removed J_arm_motor_signals1, J_arm_pots1, J_encoder_1, J_encoder_2, J_encoder_3, J_encoder_4: Conn_01x05_Socket, Connector_PinSocket_2.54mm:PinSocket_1x05_P2.54mm_Vertical, symbol Connector:Conn_01x05_Socket
- removed J_hbridge_1, J_hbridge_2, J_hbridge_3, J_hbridge_4: Conn_01x03_Socket, Connector_PinSocket_2.54mm:PinSocket_1x03_P2.54mm_Vertical, symbol Connector:Conn_01x03_Socket
- removed Q5: 2N3904, Package_TO_SOT_THT:TO-92_Inline, symbol Transistor_BJT:2N3904
- removed R18: 100k, symbol Device:R
- removed R19: 10k, symbol Device:R
- removed R4, R5, R6, R7, R8, R9: 4.7k, Resistor_THT:R_Axial_DIN0204_L3.6mm_D1.6mm_P1.90mm_Vertical, symbol Device:R
- removed R4.7k: R, Resistor_THT:R_Axial_DIN0204_L3.6mm_D1.6mm_P2.54mm_Vertical, symbol Device:R
- added C14: 1nF, Capacitor_THT:C_Disc_D5.0mm_W2.5mm_P2.50mm, symbol Device:C
- added H1, H2, H3, H4, H5, H6, H7: MountingHole, MountingHole:MountingHole_3.2mm_M3, symbol Mechanical:MountingHole
- added J1: Conn_01x02_Pin, Connector_PinHeader_2.54mm:PinHeader_1x02_P2.54mm_Vertical, symbol Connector:Conn_01x02_Pin
- added J5: Conn_01x09_Pin, Connector_PinHeader_2.54mm:PinHeader_1x09_P2.54mm_Vertical, symbol Connector:Conn_01x09_Pin
- added JP1: SolderJumper_2_Open, Jumper:SolderJumper-2_P1.3mm_Open_RoundedPad1.0x1.5mm, symbol Jumper:SolderJumper_2_Open
- added J_arm_motor_signals1: Conn_01x08_Socket, Connector_JST:JST_XH_B8B-XH-A_1x08_P2.50mm_Vertical, symbol Connector:Conn_01x08_Socket
- added J_arm_pots_1, J_encoder_1, J_encoder_2, J_encoder_3, J_encoder_4, J_hbridge_1, J_hbridge_2, J_hbridge_3, J_hbridge_4: Conn_01x04_Socket, Connector_JST:JST_XH_B4B-XH-A_1x04_P2.50mm_Vertical, symbol Connector:Conn_01x04_Socket
- added J_shift_register_extra1: Conn_01x06_Pin, Connector_PinSocket_2.54mm:PinSocket_1x06_P2.54mm_Vertical, symbol Connector:Conn_01x06_Pin
- C3: value 1nF -> 100nF
- J4: footprint Connector_PinHeader_2.54mm:PinHeader_1x02_P2.54mm_Vertical -> Project_Lib:Power_Connector
- J_i2c_1, J_i2c_2, J_i2c_3, J_ir_beac_a1, J_ir_beac_b1, J_reflectance_1: footprint Connector_PinSocket_2.54mm:PinSocket_1x05_P2.54mm_Vertical -> Connector_JST:JST_XH_B5B-XH-A_1x05_P2.50mm_Vertical
- J_switch_0, J_switch_1, J_switch_2, J_switch_3, J_switch_4, J_switch_5, J_switch_6, J_switch_7: footprint Connector_PinHeader_2.54mm:PinHeader_1x02_P2.54mm_Vertical -> Connector_JST:JST_XH_B2B-XH-A_1x02_P2.50mm_Vertical
- R1: footprint Resistor_THT:R_Axial_DIN0204_L3.6mm_D1.6mm_P2.54mm_Vertical -> Resistor_THT:R_Axial_DIN0309_L9.0mm_D3.2mm_P12.70mm_Horizontal
- R10, R11, R12, R13, R14, R15, R16, R17, R20, R21, R22, R23, R24, R25, R26, R27, R28, R29, R30, R31: footprint (none) -> Resistor_THT:R_Axial_DIN0309_L9.0mm_D3.2mm_P12.70mm_Horizontal
- R2, R3: footprint Resistor_THT:R_Axial_DIN0204_L3.6mm_D1.6mm_P1.90mm_Vertical -> Resistor_THT:R_Axial_DIN0309_L9.0mm_D3.2mm_P12.70mm_Horizontal
- U3, U6: footprint (none) -> Project_Lib:N16
- U4, U5: footprint N16 -> Project_Lib:N16
Connections:
- net +5V: now also C6.2, C7.2, C8.2, C9.2
- net 0: now also J_encoder_4.3 (Pin_3)
- net 1: now also J2.11 (Pin_11), U1.1 (gpio_1), J_hbridge_4.3 (Pin_3)
- net 10: now also J_hbridge_1.3 (Pin_3); no longer J2.11 (Pin_11), U1.1 (gpio_1)
- net 12: now also J_encoder_2.2 (Pin_2)
- net 13: now also J_encoder_2.3 (Pin_3)
- net 14: now also J_encoder_1.3 (Pin_3)
- net 15: now also J_encoder_3.2 (Pin_2)
- net 2: now also J_encoder_3.3 (Pin_3)
- net 20: now also C3.1, R2.1; no longer U3.3 (X)
- net 26: now also R3.2
- net 27: now also J_encoder_1.2 (Pin_2)
- net 3: now also J_hbridge_3.3 (Pin_3)
- net 32: now also J_arm_pots_1.2 (Pin_2)
- net 33: now also J_arm_pots_1.3 (Pin_3)
- net 37: now also J_arm_motor_signals1.6 (Pin_6)
- net 4: now also J_encoder_4.2 (Pin_2)
- net 5: now also J_arm_motor_signals1.5 (Pin_5)
- net 7: now also J_arm_motor_signals1.4 (Pin_4)
- net 8: now also J_arm_motor_signals1.2 (Pin_2)
- net 9: now also J_hbridge_2.3 (Pin_3)
- net GND: now also C10.1, C4.1, C5.1, C6.1, C7.1, C8.1, C9.1, C14.1, J_arm_motor_signals1.8 (Pin_8), J_arm_pots_1.4 (Pin_4), J_encoder_1.4 (Pin_4), J_encoder_2.4 (Pin_4), J_encoder_3.4 (Pin_4), J_encoder_4.4 (Pin_4), J_hbridge_1.4 (Pin_4), J_hbridge_2.4 (Pin_4), J_hbridge_3.4 (Pin_4), J_hbridge_4.4 (Pin_4); no longer C10.2, C4.2, C5.2, C6.2, C7.2, C8.2, C9.2
- net SHIFT_10: now also J_shift_register_extra1.1 (Pin_1); no longer R14.1
- net SHIFT_11: now also J_shift_register_extra1.2 (Pin_2); no longer R16.1
- net SHIFT_12: now also J_shift_register_extra1.3 (Pin_3)
- net SHIFT_13: now also J_shift_register_extra1.4 (Pin_4)
- net SHIFT_14: now also J_shift_register_extra1.5 (Pin_5)
- net SHIFT_15: now also J_shift_register_extra1.6 (Pin_6)
- net SHIFT_6: now also R10.1
- net SHIFT_7: now also R12.1
- net SHIFT_8: now also R14.1; no longer R10.1
- net SHIFT_9: now also R16.1; no longer R12.1
- net S_MUX_0: now also J_switch_0.2 (Pin_2), J5.1 (Pin_1); no longer C3.1, R2.1
- net S_MUX_1: now also J_switch_1.2 (Pin_2), J5.2 (Pin_2); no longer C4.1, R3.1
- net S_MUX_2: now also J_switch_2.2 (Pin_2), J5.3 (Pin_3); no longer C5.1
- net S_MUX_3: now also J_switch_3.2 (Pin_2), J5.4 (Pin_4); no longer C6.1
- net S_MUX_4: now also J_switch_4.2 (Pin_2), J5.5 (Pin_5); no longer C7.1
- net S_MUX_5: now also J_switch_5.2 (Pin_2), J5.6 (Pin_6); no longer C8.1
- net S_MUX_6: now also J_switch_6.2 (Pin_2), J5.7 (Pin_7); no longer C9.1
- net S_MUX_7: now also J_switch_7.2 (Pin_2), J5.8 (Pin_8); no longer C10.1
- net supply_3.3: now also C10.2, C4.2, C5.2, R3.1, C14.2, J1.1 (Pin_1), JP1.2 (B), J_arm_motor_signals1.7 (Pin_7), J_arm_pots_1.1 (Pin_1), J_encoder_1.1 (Pin_1), J_encoder_2.1 (Pin_1), J_encoder_3.1 (Pin_1), J_encoder_4.1 (Pin_1), J_hbridge_1.1 (Pin_1), J_hbridge_2.1 (Pin_1), J_hbridge_3.1 (Pin_1), J_hbridge_4.1 (Pin_1); no longer U2.2 (VOUT)
- net at Q9.3 (C), R27.1: now also J_hbridge_4.2 (Pin_2)
- net at Q11.3 (C), R31.1: now also J_arm_motor_signals1.3 (Pin_3)
- net at Q10.3 (C), R29.1: now also J_arm_motor_signals1.1 (Pin_1)
- net at Q6.3 (C), R21.1: now also J_hbridge_1.2 (Pin_2)
- net at Q7.3 (C), R23.1: now also J_hbridge_2.2 (Pin_2)
- net at Q8.3 (C), R25.1: now also J_hbridge_3.2 (Pin_2)
- net MUX_BYPASS: now reaches R2.2
- net MUX_BYPASS: now also U3.3 (X), J5.9 (Pin_9); no longer J_switch_0.2 (Pin_2)
- new net: J1.2 (Pin_2), JP1.1 (A), U2.2 (VOUT)
- no-connect marks 0 -> 3
Other:
- note added: "For Current Measurement"
- note added: "Shoulder Dir (pull)"
- note added: "Turntable Dir (pull)"
- note removed: "Shoulder Dir"
- note removed: "Turntable Dir"
- moved on the sheet: C1, C11, C12, D1, J_switch_0, J_switch_1, J_switch_2, J_switch_3, J_switch_4, J_switch_5, J_switch_6, J_switch_7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

Commit message: finished layout!
Parts:
- added J_debounce1: Conn_01x02_Socket, Connector_JST:JST_XH_B2B-XH-A_1x02_P2.50mm_Vertical, symbol Connector:Conn_01x02_Socket
- C10, C4, C5, C7, C8: value 1nF -> 1uF; footprint Capacitor_THT:C_Disc_D5.0mm_W2.5mm_P2.50mm -> Project_Lib:Capacitor_With_Value_uF_small
- C11, C12, C14, C6, C9: value 1nF -> 100nF; footprint Capacitor_THT:C_Disc_D5.0mm_W2.5mm_P2.50mm -> Project_Lib:Capacitor_With_Value_nF
- C3: value 100nF -> 1uF; footprint Capacitor_THT:C_Disc_D5.0mm_W2.5mm_P2.50mm -> Project_Lib:Capacitor_With_Value_uF_small
- CP1: renamed from C2; footprint Capacitor_THT:CP_Radial_D5.0mm_P2.50mm -> Project_Lib:Capacitor_With_Value_uF_small
- CP2: renamed from C1; footprint Capacitor_THT:CP_Radial_D5.0mm_P2.50mm -> Project_Lib:Capacitor_With_Value_uF_small
- CP3: renamed from C13; value 10uf -> 100uf; footprint Capacitor_THT:CP_Radial_D5.0mm_P2.50mm -> Project_Lib:Capacitor_With_Value_uF_big
- D1, D3, D4, D5, D6, D7, D8: footprint Diode_THT:D_DO-15_P5.08mm_Vertical_KathodeUp -> Project_Lib:zener_diode
- R1, R10, R11, R12, R13, R14, R15, R16, R17, R20, R21, R22, R23, R24, R25, R26, R27, R28, R29, R3, R30, R31: footprint Resistor_THT:R_Axial_DIN0309_L9.0mm_D3.2mm_P12.70mm_Horizontal -> Project_Lib:Resistor_With_Value
- R2: value 4.7k -> 1k; footprint Resistor_THT:R_Axial_DIN0309_L9.0mm_D3.2mm_P12.70mm_Horizontal -> Project_Lib:Resistor_With_Value
Connections:
- net +5V: now also C7.1, C8.1; no longer C7.2, C8.2
- net GND: now also C10.2, C4.2, C5.2, C7.2, C8.2; no longer C10.1, C4.1, C5.1, C7.1, C8.1
- net MUX_BYPASS: now also J_debounce1.2 (Pin_2); no longer R2.2
- net supply_3.3: now also C10.1, C4.1, C5.1; no longer C10.2, C4.2, C5.2
- new net: J_debounce1.1 (Pin_1), R2.2
Other:
- moved on the sheet: C10, C4, C7, C8

Commit message: finished PCB with silkscreen art! :D
Parts:
- U1: footprint Project_Lib:Untitled -> Project_Lib:ESP32_Pico_Devkit
Changed lines of the file:
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@@
 			)
 		)
-		(property "Footprint" "Project_Lib:Untitled"
+		(property "Footprint" "Project_Lib:ESP32_Pico_Devkit"
 			(at 166.37 135.89 0)
 			(effects
